File: Radar_board.sch (EAGLE design)
At the start: 22 parts, among them IC1 555, J1 AUDIO_JACK_3.5MM_PTH, U1 MAX2750AUA+

Commit message: Add files via upload
Parts:
- removed Q1: (no value), SparkFun-DiscreteSemi:TRANS_NPN_DUAL-MBT3904DW1T1
- added Q2, Q3, Q4: MMBT2222ALT1, MMBT2222ALT1:MMBT2222ALT1
- added R5, R6, R7: (no value), adafruit:R-US_R0603
- added U2: NE5532DR, NE5532DR:NE5532DR
- added X1, X2: (no value), adafruit:SMACONNECTOR_EDGE
Connections:
- new net LO_SPLIT: U$2.LO, U$4.RF1
- new net N$14: C6.1, X1.ANT
- new net N$15: J1.RSH, R5.1, U2.1OUT
- new net N$16: R5.2, R6.1, U2.1IN+
- new net PWRBIAS: L3.1, Q4.C, R7.1
- net 0: now also Q2.E, Q3.E, Q4.E, U2.VCC-, X1.GND1, X1.GND2, X1.GND3, X1.GND4, X2.GND1, X2.GND2, X2.GND3, X2.GND4; no longer Q1Q1.E, Q1Q2.E
- net LO: no longer U$2.LO, U$4.RF1
- net N$1: now also Q2.B, Q3.B, Q3.C, Q4.B; no longer Q1Q1.B, Q1Q1.C, Q1Q2.B
- net N$10: now also C3.2, X2.ANT; no longer C6.1
- net N$11: now also C5.2, U$3.RF_IN; no longer L3.1
- net N$13: now also C4.2, U$1.RF_OUT; no longer L2.1
- net N$2: now also Q2.C; no longer Q1Q2.C
- net N$7: now also L2.2, U$3.VCC2; no longer U$2.VCC, U$2.VCC@3
- net PA_IN: no longer C5.2, U$3.RF_IN
- net RFO: no longer C4.2, U$1.RF_OUT
- net TRIOUT: now also J1.TSH
- net TV_IN: now also R6.2
- net VCC3V: now also R7.2; no longer L2.2, U$3.VCC2
- net VCC6V: now also L2.1, U$2.VCC, U$2.VCC@2, U$2.VCC@3, U$2.VCC@4, U2.VCC+
Other:
- note added: "Fix me"
- moved on the sheet: C3, C4, C5, C6, J1, L1, L2, L3

Commit message: Board update and GBR files for printing
Parts:
- added IC2: TPS7A0533PDBVR, SamacSys_Parts:TPS7A0533PDBVR
Connections:
- net 0: now also IC1./RES, IC2.GND, U2.1IN-, U2.2IN+, U2.2IN-
- net VCC3V: now also IC2.OUT
- net VCC6V: now also IC2.EN, IC2.IN
Changed lines of the file:
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@@
 <setting verticaltext="up"/>
 </settings>
-<grid distance="0.1" unitdist="inch" unit="inch" style="lines" multiple="1" display="yes" altdistance="0.01" altunitdist="inch" altunit="inch"/>
+<grid distance="0.1" unitdist="inch" unit="inch" style="lines" multiple="1" display="no" altdistance="0.01" altunitdist="inch" altunit="inch"/>
 <layers>
 <layer number="1" name="Top" color="4" fill="1" visible="no" active="no"/>
@@
 <part name="X_11" library="ngspice-simulation" library_urn="urn:adsk.eagle:library:527439" deviceset="GND" device=""/>
 <part name="X_12" library="ngspice-simulation" library_urn="urn:adsk.eagle:library:527439" deviceset="GND" device=""/>
+<part name="IC2" library="SamacSys_Parts" deviceset="TPS7A0533PDBVR" device=""/>
+<part name="X_13" library="ngspice-simulation" library_urn="urn:adsk.eagle:library:527439" deviceset="GND" device=""/>
 </parts>
 <sheets>
@@
 <instance part="X_11" gate="G$1" x="472.44" y="132.08" smashed="yes"/>
 <instance part="X_12" gate="G$1" x="335.28" y="25.4" smashed="yes"/>
+<instance part="IC2" gate="G$1" x="10.16" y="177.8" smashed="yes" rot="MR0">
+<attribute name="NAME" x="-11.43" y="185.42" size="1.778" layer="95" rot="MR0" align="center-left"/>
+<attribute name="VALUE" x="-11.43" y="182.88" size="1.778" layer="96" rot="MR0" align="center-left"/>
+</instance>
+<instance part="X_13" gate="G$1" x="25.4" y="160.02" smashed="yes"/>
 </instances>
 <busses>
@@
 <wire x1="91.44" y1="66.04" x2="91.44" y2="71.12" width="0.1524" layer="91"/>
 <wire x1="73.66" y1="86.36" x2="73.66" y2="66.04" width="0.1524" layer="91"/>
-<wire x1="73.66" y1="66.04" x2="81.28" y2="66.04" width="0.1524" layer="91"/>
+<wire x1="73.66" y1="66.04" x2="76.2" y2="66.04" width="0.1524" layer="91"/>
 <junction x="91.44" y="66.04"/>
 <pinref part="C2" gate="G$1" pin="2"/>
+<wire x1="76.2" y1="66.04" x2="81.28" y2="66.04" width="0.1524" layer="91"/>
 <wire x1="81.28" y1="66.04" x2="91.44" y2="66.04" width="0.1524" layer="91"/>
 <wire x1="81.28" y1="81.28" x2="81.28" y2="66.04" width="0.1524" layer="91"/>
 <junction x="81.28" y="66.04"/>
+<pinref part="IC1" gate="G$1" pin="/RES"/>
+<wire x1="73.66" y1="99.06" x2="76.2" y2="99.06" width="0.1524" layer="91"/>
+<wire x1="76.2" y1="99.06" x2="76.2" y2="66.04" width="0.1524" layer="91"/>
+<junction x="76.2" y="66.04"/>
 </segment>
 <segment>
@@
 <segment>
 <pinref part="U2" gate="A" pin="VCC-"/>
-<wire x1="175.26" y1="157.48" x2="182.88" y2="157.48" width="0.1524" layer="91"/>
+<wire x1="175.26" y1="157.48" x2="180.34" y2="157.48" width="0.1524" layer="91"/>
+<wire x1="180.34" y1="157.48" x2="182.88" y2="157.48" width="0.1524" layer="91"/>
 <wire x1="182.88" y1="157.48" x2="182.88" y2="147.32" width="0.1524" layer="91"/>
 <pinref part="X_10" gate="G$1" pin="0"/>
+<pinref part="U2" gate="A" pin="1IN-"/>
+<wire x1="175.26" y1="172.72" x2="180.34" y2="172.72" width="0.1524" layer="91"/>
+<wire x1="180.34" y1="172.72" x2="180.34" y2="165.1" width="0.1524" layer="91"/>
+<junction x="180.34" y="157.48"/>
+<pinref part="U2" gate="A" pin="2IN+"/>
+<wire x1="180.34" y1="165.1" x2="180.34" y2="162.56" width="0.1524" layer="91"/>
+<wire x1="180.34" y1="162.56" x2="180.34" y2="157.48" width="0.1524" layer="91"/>
+<wire x1="175.26" y1="165.1" x2="180.34" y2="165.1" width="0.1524" layer="91"/>
+<junction x="180.34" y="165.1"/>
+<pinref part="U2" gate="A" pin="2IN-"/>
+<wire x1="175.26" y1="162.56" x2="180.34" y2="162.56" width="0.1524" layer="91"/>
+<junction x="180.34" y="162.56"/>
 </segment>
 <segment>
@@
 <junction x="335.28" y="30.48"/>
 </segment>
+<segment>
+<pinref part="IC2" gate="G$1" pin="GND"/>
+<wire x1="10.16" y1="175.26" x2="25.4" y2="175.26" width="0.1524" layer="91"/>
+<wire x1="25.4" y1="175.26" x2="25.4" y2="167.64" width="0.1524" layer="91"/>
+<wire x1="25.4" y1="167.64" x2="25.4" y2="160.02" width="0.1524" layer="91"/>
+<pinref part="X_13" gate="G$1" pin="0"/>
+</segment>
 </net>
 <net name="N$3" class="0">
@@
 <label x="228.6" y="172.72" size="1.778" layer="95"/>
 </segment>
+<segment>
+<pinref part="IC2" gate="G$1" pin="IN"/>
+<wire x1="10.16" y1="177.8" x2="17.78" y2="177.8" width="0.1524" layer="91"/>
+<wire x1="17.78" y1="177.8" x2="17.78" y2="180.34" width="0.1524" layer="91"/>
+<label x="17.78" y="198.12" size="1.778" layer="95"/>
+<pinref part="IC2" gate="G$1" pin="EN"/>
+<wire x1="17.78" y1="180.34" x2="17.78" y2="195.58" width="0.1524" layer="91"/>
+<wire x1="10.16" y1="172.72" x2="17.78" y2="172.72" width="0.1524" layer="91"/>
+<wire x1="17.78" y1="172.72" x2="17.78" y2="177.8" width="0.1524" layer="91"/>
+</segment>
 </net>
 <net name="TRIOUT" class="0">
@@
 <label x="0" y="114.3" size="1.778" layer="95"/>
 </segment>
+<segment>
+<pinref part="IC2" gate="G$1" pin="OUT"/>
+<wire x1="-15.24" y1="175.26" x2="-27.94" y2="175.26" width="0.1524" layer="91"/>
+<wire x1="-27.94" y1="175.26" x2="-27.94" y2="162.56" width="0.1524" layer="91"/>
+<label x="-27.94" y="157.48" size="1.778" layer="95"/>
+</segment>
 </net>

Commit message: Add files via upload
Parts:
- added C7: 0.1uF, SparkFun-Retired:.1UF-CER
- added C8: 1uF, SparkFun-Retired:.1UF-CER
- renumbered X1 to RF_INPUT, X2 to RF_OUTPUT
Connections:
- removed net 0: C2.2, IC1./RES, IC1.GND, IC2.GND, Q2.E, Q3.E, Q4.E, R4.1, RF_INPUT.GND1, RF_INPUT.GND2, RF_INPUT.GND3, RF_INPUT.GND4, RF_OUTPUT.GND1, RF_OUTPUT.GND2, RF_OUTPUT.GND3, RF_OUTPUT.GND4, U$1.@GND, U$2.GND, U$2.GND@10, U$2.GND@11, U$2.GND@2, U$2.GND@3, U$2.GND@4, U$2.GND@5, U$2.GND@6, U$2.GND@7, U$2.GND@8, U$2.GND@9, U$2.IF-, U$3.GND, U$3.GND@1, U$4.GND, U$4.GND@1, U1.GND, U1.GND@1, U2.1IN-, U2.2IN+, U2.2IN-, U2.VCC-
- new net GND: C2.2, C7.2, C8.2, IC1./RES, IC1.GND, IC2.GND, Q2.E, Q3.E, Q4.E, R4.1, RF_INPUT.GND1, RF_INPUT.GND2, RF_INPUT.GND3, RF_INPUT.GND4, RF_OUTPUT.GND1, RF_OUTPUT.GND2, RF_OUTPUT.GND3, RF_OUTPUT.GND4, U$1.@GND, U$2.GND, U$2.GND@10, U$2.GND@11, U$2.GND@2, U$2.GND@3, U$2.GND@4, U$2.GND@5, U$2.GND@6, U$2.GND@7, U$2.GND@8, U$2.GND@9, U$2.IF-, U$3.GND, U$3.GND@1, U$4.GND, U$4.GND@1, U1.GND, U1.GND@1, U2.1IN-, U2.2IN+, U2.2IN-, U2.VCC-
- net VCC3V: now also C7.1, C8.1
Changed lines of the file:
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@@
 </class>
 <class number="1" name="RF1" width="0" drill="0">
-<clearance class="1" value="0.1524"/>
+<clearance class="1" value="1.27"/>
 </class>
 </classes>
@@
 <part name="L3" library="L-07C33NJV6T" deviceset="L-07C33NJV6T" device=""/>
 <part name="U2" library="NE5532DR" deviceset="NE5532DR" device=""/>
-<part name="X1" library="adafruit" library_urn="urn:adsk.eagle:library:420" deviceset="SMACONNECTOR" device="_EDGE" package3d_urn="urn:adsk.eagle:package:6240945/1"/>
-<part name="X2" library="adafruit" library_urn="urn:adsk.eagle:library:420" deviceset="SMACONNECTOR" device="_EDGE" package3d_urn="urn:adsk.eagle:package:6240945/1"/>
+<part name="RF_INPUT" library="adafruit" library_urn="urn:adsk.eagle:library:420" deviceset="SMACONNECTOR" device="_EDGE" package3d_urn="urn:adsk.eagle:package:6240945/1"/>
+<part name="RF_OUTPUT" library="adafruit" library_urn="urn:adsk.eagle:library:420" deviceset="SMACONNECTOR" device="_EDGE" package3d_urn="urn:adsk.eagle:package:6240945/1"/>
 <part name="X_10" library="ngspice-simulation" library_urn="urn:adsk.eagle:library:527439" deviceset="GND" device=""/>
 <part name="R5" library="adafruit" library_urn="urn:adsk.eagle:library:420" deviceset="R-US_" device="R0603" package3d_urn="urn:adsk.eagle:package:6240565/1"/>
@@
 <part name="IC2" library="SamacSys_Parts" deviceset="TPS7A0533PDBVR" device=""/>
 <part name="X_13" library="ngspice-simulation" library_urn="urn:adsk.eagle:library:527439" deviceset="GND" device=""/>
+<part name="C7" library="SparkFun-Retired" library_urn="urn:adsk.eagle:library:533" deviceset=".1UF-CER" device="" value="0.1uF"/>
+<part name="C8" library="SparkFun-Retired" library_urn="urn:adsk.eagle:library:533" deviceset=".1UF-CER" device="" value="1uF"/>
+<part name="X_14" library="ngspice-simulation" library_urn="urn:adsk.eagle:library:527439" deviceset="GND" device=""/>
+<part name="X_15" library="ngspice-simulation" library_urn="urn:adsk.eagle:library:527439" deviceset="GND" device=""/>
 </parts>
 <sheets>
@@
 <attribute name="VALUE" x="161.658309375" y="147.6578" size="2.089159375" layer="96" ratio="10" rot="SMR0"/>
 </instance>
-<instance part="X1" gate="G$1" x="335.28" y="43.18" smashed="yes">
+<instance part="RF_INPUT" gate="G$1" x="335.28" y="43.18" smashed="yes">
 <attribute name="NAME" x="342.9" y="45.72" size="1.27" layer="95"/>
 <attribute name="VALUE" x="342.9" y="43.18" size="1.27" layer="95"/>
 </instance>
-<instance part="X2" gate="G$1" x="472.44" y="147.32" smashed="yes">
+<instance part="RF_OUTPUT" gate="G$1" x="472.44" y="147.32" smashed="yes">
 <attribute name="NAME" x="480.06" y="149.86" size="1.27" layer="95"/>
 <attribute name="VALUE" x="480.06" y="147.32" size="1.27" layer="95"/>
@@
 </instance>
 <instance part="X_13" gate="G$1" x="25.4" y="160.02" smashed="yes"/>
+<instance part="C7" gate="G$1" x="-17.78" y="170.18" smashed="yes">
+<attribute name="NAME" x="-16.256" y="173.101" size="1.778" layer="95"/>
+<attribute name="VALUE" x="-16.256" y="168.021" size="1.778" layer="96"/>
+</instance>
+<instance part="C8" gate="G$1" x="-30.48" y="170.18" smashed="yes">
+<attribute name="NAME" x="-28.956" y="173.101" size="1.778" layer="95"/>
+<attribute name="VALUE" x="-28.956" y="168.021" size="1.778" layer="96"/>
+</instance>
+<instance part="X_14" gate="G$1" x="-17.78" y="167.64" smashed="yes"/>
+<instance part="X_15" gate="G$1" x="-30.48" y="167.64" smashed="yes"/>
 </instances>
 <busses>
@@
 </segment>
 </net>
-<net name="0" class="0">
+<net name="GND" class="0">
 <segment>
 <wire x1="10.16" y1="71.12" x2="10.16" y2="66.04" width="0.1524" layer="91"/>
@@
 </segment>
 <segment>
-<pinref part="X2" gate="G$1" pin="GND3"/>
+<pinref part="RF_OUTPUT" gate="G$1" pin="GND3"/>
 <wire x1="469.9" y1="139.7" x2="469.9" y2="137.16" width="0.1524" layer="91"/>
-<pinref part="X2" gate="G$1" pin="GND4"/>
+<pinref part="RF_OUTPUT" gate="G$1" pin="GND4"/>
 <wire x1="469.9" y1="137.16" x2="472.44" y2="137.16" width="0.1524" layer="91"/>
 <wire x1="472.44" y1="137.16" x2="474.98" y2="137.16" width="0.1524" layer="91"/>
@@
 <wire x1="472.44" y1="137.16" x2="472.44" y2="132.08" width="0.1524" layer="91"/>
 <junction x="472.44" y="137.16"/>
-<pinref part="X2" gate="G$1" pin="GND1"/>
+<pinref part="RF_OUTPUT" gate="G$1" pin="GND1"/>
 <wire x1="469.9" y1="154.94" x2="469.9" y2="157.48" width="0.1524" layer="91"/>
 <wire x1="469.9" y1="157.48" x2="474.98" y2="157.48" width="0.1524" layer="91"/>
-<pinref part="X2" gate="G$1" pin="GND2"/>
+<pinref part="RF_OUTPUT" gate="G$1" pin="GND2"/>
 <wire x1="474.98" y1="157.48" x2="474.98" y2="154.94" width="0.1524" layer="91"/>
 <wire x1="474.98" y1="157.48" x2="485.14" y2="157.48" width="0.1524" layer="91"/>
@@
 </segment>
 <segment>
-<pinref part="X1" gate="G$1" pin="GND1"/>
+<pinref part="RF_INPUT" gate="G$1" pin="GND1"/>
 <wire x1="332.74" y1="50.8" x2="332.74" y2="55.88" width="0.1524" layer="91"/>
 <wire x1="332.74" y1="55.88" x2="337.82" y2="55.88" width="0.1524" layer="91"/>
-<pinref part="X1" gate="G$1" pin="GND2"/>
+<pinref part="RF_INPUT" gate="G$1" pin="GND2"/>
 <wire x1="337.82" y1="55.88" x2="337.82" y2="50.8" width="0.1524" layer="91"/>
 <wire x1="337.82" y1="55.88" x2="360.68" y2="55.88" width="0.1524" layer="91"/>
 <junction x="337.82" y="55.88"/>
-<pinref part="X1" gate="G$1" pin="GND3"/>
+<pinref part="RF_INPUT" gate="G$1" pin="GND3"/>
 <wire x1="332.74" y1="35.56" x2="332.74" y2="30.48" width="0.1524" layer="91"/>
 <wire x1="332.74" y1="30.48" x2="335.28" y2="30.48" width="0.1524" layer="91"/>
-<pinref part="X1" gate="G$1" pin="GND4"/>
+<pinref part="RF_INPUT" gate="G$1" pin="GND4"/>
 <wire x1="335.28" y1="30.48" x2="337.82" y2="30.48" width="0.1524" layer="91"/>
 <wire x1="337.82" y1="30.48" x2="337.82" y2="35.56" width="0.1524" layer="91"/>
@@
 <wire x1="25.4" y1="167.64" x2="25.4" y2="160.02" width="0.1524" layer="91"/>
 <pinref part="X_13" gate="G$1" pin="0"/>
+</segment>
+<segment>
+<pinref part="X_14" gate="G$1" pin="0"/>
+<pinref part="C7" gate="G$1" pin="2"/>
+</segment>
+<segment>
+<pinref part="X_15" gate="G$1" pin="0"/>
+<pinref part="C8" gate="G$1" pin="2"/>
 </segment>
 </net>
@@
 <segment>
 <pinref part="IC2" gate="G$1" pin="OUT"/>
-<wire x1="-15.24" y1="175.26" x2="-27.94" y2="175.26" width="0.1524" layer="91"/>
-<wire x1="-27.94" y1="175.26" x2="-27.94" y2="162.56" width="0.1524" layer="91"/>
-<label x="-27.94" y="157.48" size="1.778" layer="95"/>
+<wire x1="-15.24" y1="175.26" x2="-17.78" y2="175.26" width="0.1524" layer="91"/>
+<wire x1="-17.78" y1="175.26" x2="-30.48" y2="175.26" width="0.1524" layer="91"/>
+<wire x1="-30.48" y1="175.26" x2="-48.26" y2="175.26" width="0.1524" layer="91"/>
+<wire x1="-48.26" y1="175.26" x2="-48.26" y2="162.56" width="0.1524" layer="91"/>
+<label x="-48.26" y="160.02" size="1.778" layer="95"/>
+<pinref part="C7" gate="G$1" pin="1"/>
+<junction x="-17.78" y="175.26"/>
+<pinref part="C8" gate="G$1" pin="1"/>
+<junction x="-30.48" y="175.26"/>
 </segment>
 </net>
@@
 <net name="N$14" class="1">
 <segment>
-<pinref part="X1" gate="G$1" pin="ANT"/>
+<pinref part="RF_INPUT" gate="G$1" pin="ANT"/>
 <wire x1="327.66" y1="43.18" x2="243.84" y2="43.18" width="0.1524" layer="91"/>
 <pinref part="C6" gate="G$1" pin="1"/>
@@
 <net name="N$10" class="1">
 <segment>
-<pinref part="X2" gate="G$1" pin="ANT"/>
+<pinref part="RF_OUTPUT" gate="G$1" pin="ANT"/>
 <wire x1="464.82" y1="147.32" x2="439.42" y2="147.32" width="0.1524" layer="91"/>
 <pinref part="C3" gate="G$1" pin="2"/>
