File: Radar_board.brd (EAGLE design)
At the start: 160 x 100 mm, 22 parts, among them IC1 555, J1 AUDIO_JACK_3.5MM_PTH, U1 MAX2750AUA+

Commit message: Add files via upload
Parts:
- removed Q1: (no value), SparkFun-DiscreteSemi:SC70-6
- added Q2, Q3, Q4: MMBT2222ALT1, MMBT2222ALT1:SOT95P237X111-3N
- added R5, R6, R7: (no value), adafruit:R0603
- added U2: NE5532DR, NE5532DR:SOIC127P600X175-8N
- added X1, X2: (no value), adafruit:SMA_EDGELAUNCH
- moved C3 63.8 mm to (47.0, 41.9), turned to 90 degrees
- moved L3 63.0 mm to (24.1, 10.2), turned to 180 degrees
- moved L1 60.3 mm to (41.9, 33.0), turned to 270 degrees
- moved C4 59.3 mm to (44.5, 33.0), turned to 90 degrees
- moved L2 58.3 mm to (6.48, 23.7), turned to 270 degrees
- moved C6 57.8 mm to (8.89, 25.4), turned to 270 degrees
- moved C5 51.2 mm to (12.7, 19.1), turned to 180 degrees
- moved C1 50.0 mm to (36.3, 18.8)
- moved R2 48.9 mm to (36.8, 12.7), turned to 90 degrees
- moved U$4 47.7 mm to (19.1, 21.6)
- moved J1 47.5 mm to (87.6, 49.5), turned to 270 degrees
- moved R3 44.3 mm to (36.1, 16.9), turned to 180 degrees
- moved D1 43.1 mm to (23.2, 28.6)
- moved R4 42.8 mm to (13.3, 25.1), turned to 180 degrees
- moved R1 38.0 mm to (23.2, 32.4), turned to 180 degrees
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Connections:
- new net LO_SPLIT: U$2.11, U$4.1
- new net N$14: C6.1, X1.P
- new net N$15: J1.RSH, R5.1, U2.1
- new net N$16: R5.2, R6.1, U2.3
- new net PWRBIAS: L3.1, Q4.3, R7.1
- net 0: now also Q2.2, Q3.2, Q4.2, U2.4, X1.GND@1, X1.GND@2, X1.GND@3, X1.GND@4, X2.GND@1, X2.GND@2, X2.GND@3, X2.GND@4; no longer Q1.1, Q1.4
- net LO: no longer U$2.11, U$4.1
- net N$1: now also Q2.1, Q3.1, Q3.3, Q4.1; no longer Q1.2, Q1.3, Q1.5
- net N$10: now also C3.2, X2.P; no longer C6.1
- net N$11: now also C5.2, U$3.1; no longer L3.1
- net N$13: now also C4.2, U$1.6; no longer L2.1
- net N$2: now also Q2.3; no longer Q1.6
- net N$7: now also L2.2, U$3.5; no longer U$2.1, U$2.8
- net PA_IN: no longer C5.2, U$3.1
- net RFO: no longer C4.2, U$1.6
- net TRIOUT: now also J1.TSH
- net TV_IN: now also R6.2
- net VCC3V: now also R7.2; no longer L2.2, U$3.5
- net VCC6V: now also L2.1, U$2.1, U$2.14, U$2.6, U$2.8, U2.8
Routing:
- net N$15: track 0.00 -> 77.1 mm
- net N$1: track 0.00 -> 44.1 mm
- net VCC6V: track 0.00 -> 34.5 mm, vias 0 -> 6
- net TRIOUT: track 0.00 -> 31.9 mm, vias 0 -> 4
- net VCC1V: track 0.00 -> 31.8 mm, vias 0 -> 2
- net LO_SPLIT: track 0.00 -> 23.7 mm
- net N$14: track 0.00 -> 22.5 mm
- net N$2: track 0.00 -> 21.9 mm
- net N$16: track 0.00 -> 21.7 mm
- net N$5: track 0.00 -> 14.9 mm
- net VCC3V: track 0.00 -> 14.0 mm, vias 0 -> 3
- net PWRBIAS: track 0.00 -> 12.5 mm
- net RFO: track 0.00 -> 10.2 mm
- net N$8: track 0.00 -> 6.06 mm
- net N$4: track 0.00 -> 6.01 mm
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- added copper zone on layer 1, net 0
- added copper zone on layer 16, net GND
- added copper zone on layer 16, net TRIOUT
- added copper zone on layer 16, net VCC3V
- added copper zone on layer 16, net VCC6V
Other:
- board size 160 x 100 mm -> 97.8 x 53 mm

Commit message: Board update and GBR files for printing
Parts:
- added IC2: TPS7A0533PDBVR, SamacSys_Parts:SOT95P280X145-5N
Connections:
- net 0: now also IC1.4, IC2.2, U2.2, U2.5, U2.6
- net VCC3V: now also IC2.5
- net VCC6V: now also IC2.1, IC2.3
Routing:
- net VCC3V: track 14.0 -> 18.0 mm
- added copper zone on layer 1, net VCC6V
Other:
- board size 97.8 x 53 mm -> 97.8 x 53.4 mm
Changed lines of the file:
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@@
 <plain>
 <wire x1="0" y1="0" x2="97.77" y2="0" width="0" layer="20"/>
-<wire x1="97.77" y1="0" x2="97.77" y2="53.01" width="0" layer="20"/>
-<wire x1="97.77" y1="53.01" x2="0" y2="53.01" width="0" layer="20"/>
-<wire x1="0" y1="53.01" x2="0" y2="0" width="0" layer="20"/>
+<wire x1="97.77" y1="0" x2="97.77" y2="53.391" width="0" layer="20"/>
+<wire x1="97.77" y1="53.391" x2="0" y2="53.264" width="0" layer="20"/>
+<wire x1="0" y1="53.264" x2="0" y2="0" width="0" layer="20"/>
 </plain>
 <attributes>
@@
 <attribute name="VALUE" x="31.242" y="11.811" size="1.27" layer="27" rot="R90"/>
 </element>
+<element name="IC2" library="SamacSys_Parts" package="SOT95P280X145-5N" value="TPS7A0533PDBVR" x="24.13" y="15.24" smashed="yes">
+<attribute name="DESCRIPTION" value="1-A, ultra-low-IQ, 200-mA low-dropout (LDO) regulator in a small-sized package" x="24.13" y="15.24" size="1.778" layer="27" display="off"/>
+<attribute name="HEIGHT" value="1.45mm" x="24.13" y="15.24" size="1.778" layer="27" display="off"/>
+<attribute name="MANUFACTURER_NAME" value="Texas Instruments" x="24.13" y="15.24" size="1.778" layer="27" display="off"/>
+<attribute name="MANUFACTURER_PART_NUMBER" value="TPS7A0533PDBVR" x="24.13" y="15.24" size="1.778" layer="27" display="off"/>
+<attribute name="MOUSER_PART_NUMBER" value="595-TPS7A0533PDBVR" x="24.13" y="15.24" size="1.778" layer="27" display="off"/>
+<attribute name="MOUSER_PRICE-STOCK" value="https://www.mouser.com/Search/Refine.aspx?Keyword=595-TPS7A0533PDBVR" x="24.13" y="15.24" size="1.778" layer="27" display="off"/>
+<attribute name="NAME" x="21.59" y="10.16" size="1.27" layer="25" align="center"/>
+<attribute name="VALUE" x="13.97" y="15.24" size="1.27" layer="27" align="center"/>
+</element>
 </elements>
 <signals>
@@
 <wire x1="28.073" y1="21.28" x2="28.234" y2="21.441" width="0.2032" layer="1"/>
 <wire x1="28.234" y1="21.441" x2="28.75055" y2="21.441" width="0.2032" layer="1"/>
-<polygon width="0.1524" layer="1">
-<vertex x="162.56" y="104.14"/>
-<vertex x="165.1" y="101.6"/>
-<vertex x="165.1" y="-3.81"/>
-<vertex x="0" y="-3.81"/>
-<vertex x="-8.89" y="5.08"/>
-<vertex x="-8.89" y="95.25"/>
-<vertex x="0" y="104.14"/>
+<polygon width="0.1524" layer="1" rank="2">
+<vertex x="97.79" y="53.34"/>
+<vertex x="97.79" y="0"/>
+<vertex x="0" y="0"/>
+<vertex x="0" y="53.34"/>
 </polygon>
 <contactref element="X2" pad="GND@2"/>
@@
 <contactref element="X1" pad="GND@2"/>
 <contactref element="X1" pad="GND@1"/>
+<contactref element="IC1" pad="4"/>
+<contactref element="U2" pad="2"/>
+<contactref element="U2" pad="6"/>
+<contactref element="U2" pad="5"/>
+<contactref element="IC2" pad="2"/>
 <wire x1="49.53" y1="48.768" x2="49.53" y2="48.768" width="0" layer="19" extent="1-16"/>
 <wire x1="44.45" y1="48.768" x2="44.45" y2="48.768" width="0" layer="19" extent="1-16"/>
@@
 <wire x1="34.4677" y1="27.94" x2="34.4677" y2="26.64" width="0" layer="19" extent="1-1"/>
 <wire x1="34.4677" y1="28.59" x2="34.4677" y2="27.94" width="0" layer="19" extent="1-1"/>
+<wire x1="53.2638" y1="29.845" x2="53.2638" y2="32.385" width="0" layer="19" extent="1-1"/>
+<wire x1="12.44" y1="27.305" x2="14.185" y2="25.146" width="0" layer="19" extent="1-1"/>
 <wire x1="23.743" y1="19.98" x2="20.2956" y2="22.54" width="0" layer="19" extent="1-1"/>
 <wire x1="28.073" y1="21.28" x2="23.743" y2="19.98" width="0" layer="19" extent="1-1"/>
+<wire x1="22.88" y1="15.24" x2="23.743" y2="19.98" width="0" layer="19" extent="1-1"/>
+<wire x1="48.3362" y1="32.385" x2="53.2638" y2="32.385" width="0" layer="19" extent="1-1"/>
+<wire x1="48.3362" y1="31.115" x2="48.3362" y2="32.385" width="0" layer="19" extent="1-1"/>
 <wire x1="9.7087" y1="21.332" x2="14.185" y2="25.146" width="0" layer="19" extent="1-1"/>
 <wire x1="9.7087" y1="20.832" x2="9.7087" y2="21.332" width="0" layer="19" extent="1-1"/>
@@
 <vertex x="16.51" y="34.29"/>
 </polygon>
+<contactref element="IC2" pad="1"/>
+<contactref element="IC2" pad="3"/>
+<polygon width="0.254" layer="1">
+<vertex x="20.32" y="17.78"/>
+<vertex x="24.13" y="17.78"/>
+<vertex x="24.13" y="12.7"/>
+<vertex x="3.81" y="12.7"/>
+<vertex x="2.54" y="13.97"/>
+<vertex x="2.54" y="26.289"/>
+<vertex x="6.35" y="26.289"/>
+<vertex x="6.35" y="24.892"/>
+<vertex x="4.318" y="24.892"/>
+<vertex x="4.318" y="16.51"/>
+<vertex x="19.05" y="16.51"/>
+</polygon>
 <wire x1="38.13" y1="30.3023" x2="39.1923" y2="26.64" width="0" layer="19" extent="1-1"/>
 </signal>
@@
 <vertex x="6.35" y="31.75"/>
 </polygon>
+<contactref element="IC2" pad="5"/>
+<wire x1="25.38" y1="16.19" x2="28.89" y2="16.19" width="0.508" layer="1"/>
+<wire x1="28.89" y1="16.19" x2="29.21" y2="16.51" width="0.508" layer="1"/>
 <wire x1="36.83" y1="13.55" x2="29.21" y2="13.55" width="0" layer="19" extent="1-1"/>
 </signal>
@@
 <signal name="GND">
 <polygon width="0.2032" layer="16" rank="4">
-<vertex x="-2.54" y="55.88"/>
-<vertex x="104.14" y="55.88"/>
-<vertex x="106.68" y="53.34"/>
-<vertex x="106.68" y="10.16"/>
-<vertex x="92.71" y="-3.81"/>
-<vertex x="-2.54" y="-3.81"/>
+<vertex x="0" y="53.34"/>
+<vertex x="97.79" y="53.34"/>
+<vertex x="97.79" y="0"/>
+<vertex x="0" y="0"/>
 </polygon>
 </signal>

Commit message: Add files via upload
Parts:
- removed X1, X2: (no value), adafruit:SMA_EDGELAUNCH
- added C7: 0.1uF, SparkFun-Retired:0402-CAP
- added C8: 1uF, SparkFun-Retired:0402-CAP
- added RF_INPUT, RF_OUTPUT: (no value), adafruit:SMA_EDGELAUNCH
- moved J1 54.3 mm to (58.4, 3.81), turned to 90 degrees
- moved C6 16.4 mm to (8.89, 41.8)
- moved C3 4.07 mm to (42.9, 42.0)
Connections:
- removed net 0: C2.2, IC1.1, IC1.4, IC2.2, Q2.2, Q3.2, Q4.2, R4.1, U$1.7, U$2.10, U$2.12, U$2.13, U$2.15, U$2.16, U$2.17, U$2.18, U$2.20, U$2.21, U$2.3, U$2.4, U$2.5, U$2.9, U$3.2, U$3.3, U$3.9, U$4.2, U$4.5, U1.3, U1.8, U2.2, U2.4, U2.5, U2.6, X1.GND@1, X1.GND@2, X1.GND@3, X1.GND@4, X2.GND@1, X2.GND@2, X2.GND@3, X2.GND@4
- new net GND: C2.2, C7.2, C8.2, IC1.1, IC1.4, IC2.2, Q2.2, Q3.2, Q4.2, R4.1, RF_INPUT.GND@1, RF_INPUT.GND@2, RF_INPUT.GND@3, RF_INPUT.GND@4, RF_OUTPUT.GND@1, RF_OUTPUT.GND@2, RF_OUTPUT.GND@3, RF_OUTPUT.GND@4, U$1.7, U$2.10, U$2.12, U$2.13, U$2.15, U$2.16, U$2.17, U$2.18, U$2.20, U$2.21, U$2.3, U$2.4, U$2.5, U$2.9, U$3.2, U$3.3, U$3.9, U$4.2, U$4.5, U1.3, U1.8, U2.2, U2.4, U2.5, U2.6
- net N$10: now also RF_OUTPUT.P; no longer X2.P
- net N$14: now also RF_INPUT.P; no longer X1.P
- net VCC3V: now also C7.1, C8.1
Routing:
- net GND: track 0.00 -> 51.0 mm, vias 0 -> 3
- net N$15: track 77.1 -> 32.8 mm
- net N$14: track 22.5 -> 3.59 mm
- net N$12: track 4.13 -> 20.5 mm
- net VCC3V: track 18.0 -> 25.6 mm
- net N$10: track 6.01 -> 1.56 mm
- net N$8: track 6.06 -> 2.94 mm
- net 0: track 3.03 -> 0.00 mm
- net VCC6V: track 34.5 -> 32.0 mm, vias 6 -> 5
- net N$17: track 0.00 -> 2.54 mm, vias 0 -> 1
- net TRIOUT: track 31.9 -> 29.8 mm, vias 4 -> 5
- net LO_SPLIT: track 23.7 -> 22.6 mm
- net PA_IN: track 5.84 -> 4.75 mm
- added copper zone on layer 1, net GND
- added copper zone on layer 15, net GND
- added copper zone on layer 15, net TRIOUT
- added copper zone on layer 15, net VCC3V
- added copper zone on layer 15, net VCC6V
- removed copper zone on layer 1, net 0
- removed copper zone on layer 16, net GND
- removed copper zone on layer 16, net TRIOUT
- removed copper zone on layer 16, net VCC3V
- removed copper zone on layer 16, net VCC6V
Other:
- board size 97.8 x 53.4 mm -> 66 x 50.2 mm

Commit message: Add files via upload
Routing:
- net VCC6V: track 32.0 -> 34.5 mm, vias 5 -> 6
- net N$17: track 2.54 -> 0.00 mm, vias 1 -> 0
- net GND: vias 3 -> 4
- added copper zone on layer 16, net GND
- added copper zone on layer 2, net GND
Changed lines of the file:
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@@
 <layers>
 <layer number="1" name="Top" color="4" fill="1" visible="yes" active="yes"/>
-<layer number="2" name="Route2" color="16" fill="1" visible="no" active="yes"/>
+<layer number="2" name="Route2" color="16" fill="1" visible="yes" active="yes"/>
 <layer number="3" name="Route3" color="17" fill="1" visible="no" active="no"/>
 <layer number="4" name="Route4" color="18" fill="1" visible="no" active="no"/>
@@
 <wire x1="38.1" y1="31.75" x2="38.1" y2="32.99" width="0.381" layer="1"/>
 <wire x1="38.1" y1="32.99" x2="38.13" y2="33.02" width="0.381" layer="1"/>
+<via x="1.27" y="14.605" extent="1-16" drill="0.635"/>
+<wire x1="1.27" y1="14.605" x2="2.54" y2="14.605" width="1.27" layer="1"/>
+<wire x1="2.54" y1="14.605" x2="3.81" y2="14.605" width="1.27" layer="1"/>
 <wire x1="39.37" y1="26.368" x2="39.1923" y2="26.64" width="0" layer="19" extent="1-1"/>
 <wire x1="38.13" y1="30.3023" x2="39.1923" y2="26.64" width="0" layer="19" extent="1-1"/>
@@
 <wire x1="1.27" y1="10.16" x2="3.81" y2="10.16" width="1.27" layer="1"/>
 <via x="35.56" y="1.27" extent="1-16" drill="0.635"/>
-<wire x1="45.466" y1="46.101" x2="45.466" y2="46.101" width="0" layer="19" extent="1-16"/>
-<wire x1="40.386" y1="46.101" x2="40.386" y2="46.101" width="0" layer="19" extent="1-16"/>
-<wire x1="11.43" y1="46.228" x2="11.43" y2="46.228" width="0" layer="19" extent="1-16"/>
-<wire x1="6.35" y1="46.228" x2="6.35" y2="46.228" width="0" layer="19" extent="1-16"/>
+<polygon width="0.1524" layer="2">
+<vertex x="0" y="50.8"/>
+<vertex x="66.04" y="50.8"/>
+<vertex x="66.04" y="0"/>
+<vertex x="0" y="0"/>
+</polygon>
+<polygon width="0.1524" layer="16">
+<vertex x="0" y="50.8"/>
+<vertex x="66.04" y="50.8"/>
+<vertex x="66.04" y="0"/>
+<vertex x="0" y="0"/>
+</polygon>
+<via x="60.96" y="44.45" extent="1-16" drill="0.635"/>
+<wire x1="48.3362" y1="32.385" x2="42.922" y2="36.9003" width="0" layer="19" extent="1-1"/>
 <wire x1="9.7087" y1="20.832" x2="9.7087" y2="21.332" width="0" layer="19" extent="1-1"/>
 <wire x1="39.1923" y1="28.59" x2="39.1923" y2="29.24" width="0" layer="19" extent="1-1"/>
@@
 <wire x1="27.051" y1="12.05" x2="31.75" y2="12.05" width="0" layer="19" extent="1-1"/>
 <wire x1="22.88" y1="15.24" x2="23.743" y2="19.98" width="0" layer="19" extent="1-1"/>
-<wire x1="42.922" y1="36.9003" x2="48.3362" y2="32.385" width="0" layer="19" extent="1-1"/>
-</signal>
-<signal name="N$17">
-<via x="1.27" y="14.605" extent="1-16" drill="0.635"/>
-<wire x1="1.27" y1="14.605" x2="2.54" y2="14.605" width="1.27" layer="1"/>
-<wire x1="2.54" y1="14.605" x2="3.81" y2="14.605" width="1.27" layer="1"/>
 </signal>
 </signals>
